File: Eval Board.kicad_pcb (KiCad board)
At the start: 2 copper layers, 50.8 x 33.5 mm, 34 parts, among them J1 I OUT, J2 Q OUT, J3 LO, J4 RF, U1 LTC5584

Commit message: Rev 0.1
Parts:
- moved C16 0.52 mm to (179.5, 72.8)
